File: pcb/ADC/ADC.brd (EAGLE design)
At the start: 22.4 x 30 mm, 15 parts, among them IC1 AD7997BRU, IC2 MCP1700

Commit message: Pridana dokumentace modulu ADC RevB
Parts:
- IC2: value MCP1700 -> MCP1700T3302ETT
Changed lines of the file:
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@@
 <attribute name="VALUE" x="3.81" y="14.605" size="0.6096" layer="27" rot="R270"/>
 </element>
-<element name="IC2" library="!stab" package="SOT23" value="MCP1700" x="17.78" y="1.905" rot="R180"/>
+<element name="IC2" library="!stab" package="SOT23" value="MCP1700T3302ETT" x="17.78" y="1.905" smashed="yes" rot="R180">
+<attribute name="NAME" x="17.78" y="1.905" size="0.6096" layer="25" rot="R180" align="center"/>
+<attribute name="VALUE" x="20.32" y="-0.635" size="0.6096" layer="27" rot="R270" align="center"/>
+</element>
 <element name="C2" library="!discrete" package="0805" value="1M" x="13.335" y="-2.54" rot="R270">
 <attribute name="VOLTAGE" value="16V" x="13.335" y="-2.54" size="0.635" layer="27" font="vector" rot="R270" display="off"/>

Commit message: Aktualizovany partlisty u obou modulu KM2 i ADC. Odkazy a ceny jsou uvnitr schematu.
Parts:
- D1: value KP-2012ID -> KP-2012SGC
- R3: value 850 -> 270
Changed lines of the file:
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@@
 <setting verticaltext="up"/>
 </settings>
-<grid distance="25" unitdist="mil" unit="mm" style="lines" multiple="4" display="yes" altdistance="5" altunitdist="mil" altunit="mil"/>
+<grid distance="25" unitdist="mil" unit="mil" style="lines" multiple="4" display="yes" altdistance="5" altunitdist="mil" altunit="mil"/>
 <layers>
 <layer number="1" name="Top" color="4" fill="1" visible="yes" active="yes"/>
@@
 </autorouter>
 <elements>
-<element name="IC1" library="!ic_analogdevices" package="TSSOP20" value="AD7997BRU" x="6.985" y="0" rot="R180"/>
-<element name="JP3" library="!pinhead" package="1X04_250_MX5268" value="MX-5268-04A" x="15.24" y="8.255" rot="MR180"/>
+<element name="IC1" library="!ic_analogdevices" package="TSSOP20" value="AD7997BRU" x="6.985" y="0" rot="R180">
+<attribute name="PRICE" value="69.00" x="6.985" y="0" size="1.778" layer="27" rot="R180" display="off"/>
+<attribute name="URL" value="https://www.gme.cz/ad7997bruz-0-tssop20-analog-devices" x="6.985" y="0" size="1.778" layer="27" rot="R180" display="off"/>
+</element>
+<element name="JP3" library="!pinhead" package="1X04_250_MX5268" value="MX-5268-04A" x="15.24" y="8.255" rot="MR180">
+<attribute name="PRICE" value="2.52" x="15.24" y="8.255" size="1.778" layer="28" rot="MR180" display="off"/>
+<attribute name="URL" value="http://www.tme.eu/cz/details/mx-5268-04a/signalove-konektory-raster-250mm/molex/022057045-22-05-7045-5268-04a/" x="15.24" y="8.255" size="1.778" layer="28" rot="MR180" display="off"/>
+</element>
 <element name="C1" library="!discrete" package="0805" value="1M" x="13.335" y="1.905" rot="R90">
 <attribute name="VOLTAGE" value="16V" x="13.335" y="1.905" size="0.635" layer="27" font="vector" rot="R90" display="off"/>
 <attribute name="MATERIAL" value="X7R" x="13.335" y="1.905" size="0.635" layer="27" font="vector" rot="R90" display="off"/>
+<attribute name="PRICE" value="0.27" x="13.335" y="1.905" size="1.778" layer="27" rot="R90" display="off"/>
+<attribute name="URL" value="http://www.tme.eu/cz/details/cl21b105kofnnng/kondenzatory-mlcc-smd-0805/samsung/" x="13.335" y="1.905" size="1.778" layer="27" rot="R90" display="off"/>
 </element>
 <element name="R1" library="!discrete" package="0805" value="DNP" x="11.43" y="-2.54" rot="R270">
@@
 <attribute name="NAME" x="4.445" y="-14.605" size="0.6096" layer="25" ratio="10" rot="R90"/>
 <attribute name="VALUE" x="3.81" y="14.605" size="0.6096" layer="27" rot="R270"/>
+<attribute name="PRICE" value="2.80" x="0" y="-1.27" size="1.778" layer="27" rot="R90" display="off"/>
+<attribute name="URL" value="http://www.tme.eu/cz/details/zl201-14g/konektory-hrebinky/connfly/ds1021-1_14sf11/" x="0" y="-1.27" size="1.778" layer="27" rot="R90" display="off"/>
 </element>
 <element name="IC2" library="!stab" package="SOT23" value="MCP1700T3302ETT" x="17.78" y="1.905" smashed="yes" rot="R180">
 <attribute name="NAME" x="17.78" y="1.905" size="0.6096" layer="25" rot="R180" align="center"/>
 <attribute name="VALUE" x="20.32" y="-0.635" size="0.6096" layer="27" rot="R270" align="center"/>
+<attribute name="PRICE" value="8.78" x="17.78" y="1.905" size="1.778" layer="27" rot="R180" display="off"/>
+<attribute name="URL" value="http://www.tme.eu/cz/details/mcp1700t3302ett/stabilizatory-napeti-neregulovane-ldo/microchip-technology/mcp1700t-3302ett/" x="17.78" y="1.905" size="1.778" layer="27" rot="R180" display="off"/>
 </element>
 <element name="C2" library="!discrete" package="0805" value="1M" x="13.335" y="-2.54" rot="R270">
 <attribute name="VOLTAGE" value="16V" x="13.335" y="-2.54" size="0.635" layer="27" font="vector" rot="R270" display="off"/>
 <attribute name="MATERIAL" value="X7R" x="13.335" y="-2.54" size="0.635" layer="27" font="vector" rot="R270" display="off"/>
-</element>
-<element name="JP2" library="!pinhead" package="1X04_250_MX5268" value="MX-5268-04A" x="15.24" y="-8.255" rot="MR0"/>
-<element name="D1" library="!opto" package="LED_0805" value="KP-2012ID" x="15.24" y="-2.54" smashed="yes" rot="R270">
+<attribute name="PRICE" value="0.27" x="13.335" y="-2.54" size="1.778" layer="27" rot="R270" display="off"/>
+<attribute name="URL" value="http://www.tme.eu/cz/details/cl21b105kofnnng/kondenzatory-mlcc-smd-0805/samsung/" x="13.335" y="-2.54" size="1.778" layer="27" rot="R270" display="off"/>
+</element>
+<element name="JP2" library="!pinhead" package="1X04_250_MX5268" value="MX-5268-04A" x="15.24" y="-8.255" rot="MR0">
+<attribute name="PRICE" value="2.52" x="15.24" y="-8.255" size="1.778" layer="28" rot="MR0" display="off"/>
+<attribute name="URL" value="http://www.tme.eu/cz/details/mx-5268-04a/signalove-konektory-raster-250mm/molex/022057045-22-05-7045-5268-04a/" x="15.24" y="-8.255" size="1.778" layer="28" rot="MR0" display="off"/>
+</element>
+<element name="D1" library="!opto" package="LED_0805" value="KP-2012SGC" x="15.24" y="-2.54" smashed="yes" rot="R270">
 <attribute name="NAME" x="15.24" y="-3.81" size="0.6096" layer="25" align="center"/>
 <attribute name="VALUE" x="16.51" y="-2.54" size="0.6096" layer="27" rot="R270" align="center"/>
-</element>
-<element name="R3" library="!discrete" package="0805" value="850" x="15.24" y="1.905" rot="R90">
+<attribute name="PRICE" value="1.00" x="15.24" y="-2.54" size="1.778" layer="27" rot="R270" display="off"/>
+<attribute name="URL" value="http://www.tme.eu/cz/details/kp-2012sgc/diody-led-smd-barevne/kingbright-electronic/" x="15.24" y="-2.54" size="1.778" layer="27" rot="R270" display="off"/>
+</element>
+<element name="R3" library="!discrete" package="0805" value="270" x="15.24" y="1.905" rot="R90">
 <attribute name="TOLERANCE" value="" x="15.24" y="1.905" size="2.1844" layer="27" font="vector" rot="R90" display="off"/>
+<attribute name="PRICE" value="0.15" x="15.24" y="1.905" size="1.778" layer="27" rot="R90" display="off"/>
+<attribute name="URL" value="http://www.tme.eu/cz/details/rc0805jr-07270r/rezistory-smd-0805/yageo/rc0805jr-07270rl/" x="15.24" y="1.905" size="1.778" layer="27" rot="R90" display="off"/>
 </element>
 <element name="U$2" library="!frames" package="DIN_A4_SCALE4" value="" x="-12.7" y="-43.18"/>
