File: pcb/MAINBOARD/MAINBOARD.sch (EAGLE design)
At the start: 67 parts, among them Q1 20MHz, SW1 P-DT6E, SW2 P-DT6E, T1 IRMLM0060TRPbF

Commit message: Přidány opravy chyb, které se vyskytly během oživování
Parts:
- added C10, C7: 100n, !discrete:C0805
- added C8, C9: 1n, !discrete:C0805
- added D7: 1N4148, #PaJa_30:1N4148_SOD80
- added R20, R21: 100k, !discrete:R_R0805
- C1, C3: value 100uF/16V -> 100uF; VOLTAGE (none) -> 16V
- C2, C5: VOLTAGE 16V -> 50V
- D2, D3, D4, D5, D6: device led:LEDCHIPLED_0805 -> !opto:LED0805
- DC1: value DC-DC-STEPDOWN -> MP1584; PRICE 15 -> 13; URL nekde na ebay -> https://www.aliexpress.com/item/Free-Shipping-200PCS-MP1584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
- DZ1: value D -ZENEROVA 3.3V -> BZV55C3.3; URL http://www.tme.eu/cz/details/bzv55-c3v6.115/zenerovy-diody-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 -> http://www.tme.eu/cz/details/tzmc3v3-gs08/zenerovy-diody-sm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
- DZ2: value D-ZENEROVA 3.3V -> BZV55C3.3; URL http://www.tme.eu/cz/details/bzv55-c3v6.115/zenerovy-diody-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 -> http://www.tme.eu/cz/details/tzmc3v3-gs08/zenerovy-diody-sm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
- R1, R11, R3, R7: device rcl:R-EU_R0603 -> !discrete:R_R0805; PRICE (none) -> 0.5; TOLERANCE (none) -> 1%; URL (none) -> http://www.tme.eu/cz/details/hp05-470r1%25/rezistory-smd-08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
- R10, R14, R16, R17, R18, R19: value 68R -> 330R; PRICE 0.15 -> 0.22; TOLERANCE (none) -> 1%; URL http://www.tme.eu/cz/details/rc0805jr-07270r/rezistory-smd-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 -> http://www.tme.eu/cz/details/smd0805-330r-1%25/rezistory-sm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
- R12, R2, R4, R8: device rcl:R-EU_R0603 -> !discrete:R_R0805; PRICE (none) -> 0.22; TOLERANCE (none) -> 1%; URL (none) -> http://www.tme.eu/cz/details/smd0805-330r-1%25/rezistory-sm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
- R13: TOLERANCE (none) -> 5%
- R15: PRICE 0.15 -> 0.22; TOLERANCE (none) -> 1%; URL http://www.tme.eu/cz/details/rc0805jr-07270r/rezistory-smd-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 -> http://www.tme.eu/cz/details/rc0805fr-072k7/rezistory-smd-0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
- R5: device rcl:R-EU_M1206 -> !discrete:R_R1206; TOLERANCE (none) -> 5%
- R6, R9: value DNP -> 10k; PRICE (none) -> 0.15; TOLERANCE (none) -> 5%; URL (none) -> http://www.tme.eu/cz/details/rc0805jr-07510k/rezistory-smd-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
- T1: device transistor:-NPN-SOT23-EBC -> #TD:NPNBCE; PRICE 1 -> 0.5; URL nejaky NPN -> http://www.tme.eu/cz/details/bc817-16-dio/tranzistory-npn-s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
Connections:
- net N$2 renamed B
- removed net N$13: D3.C, R17.2
- removed net N$15: D5.C, R18.2
- removed net N$9: D2.C, R16.2
- new net C: D7.A, SG1.-, T1.C
- new net N$2: D6.A, R19.2
- new net N$7: D2.A, R16.2
- net +3V3: now also C10.2, C9.2, R20.2, R21.2; no longer D2.A, D3.A, D4.A, D5.A, D6.A, SG1.+
- net +5V: now also C7.1, C8.1, D7.K, SG1.+
- net AGND: no longer D1.C
- net GND: now also C10.1, C7.2, C8.2, C9.1, D1.C, D2.C, D3.C, D4.C, D5.C, D6.C
- net GPB5-2: now also R20.1
- net GPB6-2: now also R21.1
- net N$3: now also D3.A, R17.2; no longer SG1.-, T1.C
- net N$4: now also D4.A, R14.2; no longer D6.C, R19.2
- net N$6: now also D5.A, R18.2; no longer D4.C, R14.2
Other:
- note added: "GPIO adresa na I2C 0x20"
- note added: "adresa 0x21 musi byt odpor"
- note added: "adresa 0x22 musi byt odpor"
- note added: "dimenzovano na 5mA"
- moved on the sheet: ARK1, B1, C1, C2, C3, C4, C5, C6, DZ1, DZ2, F1, IO1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

Commit message: Velke upravy pred odeslanim do seriove vyroby
Parts:
- removed DZ1, DZ2: BZV55C3.3, #PaJa_22:D-ZENEROVA_0,5W_BZV55C_SMD
- removed T1: IRMLM0060TRPbF, #TD:NPNBCE
- added D8: BZV55C3.3, !discrete:D_ZENER_SOD80
- added D9: BZV55V3.3, !discrete:D_ZENER_SOD80
- added T2: (no value), !transistor:_EMOS_N_SOT23_GDS
- D7: value 1N4148 -> LL4148; device #PaJa_30:1N4148_SOD80 -> !diody:D_SOD80; PRICE 0.45 -> (none); URL http://www.tme.eu/cz/details/ll4148-dio/univerzalni-diody-s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 -> (none)
Connections:
- net B: now also T2.G; no longer T1.B
- net C: now also T2.D; no longer T1.C
- net GND: now also D8.A, D9.A, T2.S; no longer DZ1.A, DZ2.A, T1.E
- net SCL: now also D9.K; no longer DZ2.K
- net SDA: now also D8.K; no longer DZ1.K

Commit message: New version of board, shipped to SeedStudio (2x KM2-B, 1x Mainboard -A)
Parts:
- removed ARK1: ARK500/2, #TD:ARK500/2
- removed IO1: ATmega88PA-AU, !ic_avr:MEGA8
- removed IO4: MCP23017SO, microchip:MCP23017SO
- removed IO5: LD1086, #TD:STABI_DPACK
- removed JP14, JP23, JP24, JP28, JP29: S1G8_JUM, #Lamacie lišty by TD:S1G8_JUM
- removed Q1: 20MHz, crystal:CRYSTALHC49S
- added C11: 22M, !discrete:CECT7343
- added C12: 100n, !discrete:C0805
- added D10, D11, D12, D13, D14, D15, D16, D17, D18, D19, D20, D21, D22, D23, D24, D25, D26, D27: KP-2012SGC, !opto:LED0805
- added D28: SK24, !discrete:D_SMB
- added IC1: PCA9685, !ic_nxp:PCA9685
- added IC2: MCP23017/SO, !ic_microchip:MCP23017/SO
- added IC3: ULN2003D1013TR, !uln:ULN200X_SO
- added IC4: LD1086DT33, !stab:LD1086
- added JP12: DS1021-1*8SF1-1, !pinhead:PINHD-1X7
- added JP13: TB-5.08-P-2P/BL, !pinhead:PINHD-1X2_508_SROUB
- added R22, R23, R24, R25, R26, R27, R28, R29, R30: 330, !discrete:R_R0805
- C1: value 100uF -> 100n; device rcl:CPOL-EUE5-10.5 -> !discrete:C0805; PRICE 1.3 -> 0.16; URL http://www.tme.eu/cz/details/uvz1c101mdd/elektrolyticke-kon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 -> http://www.tme.eu/cz/details/cc0805krx7r9104/kondenzatory-m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; VOLTAGE 16V -> 50V
- C3: value 100uF -> 22M; device rcl:CPOL-EUE5-10.5 -> !discrete:CECT7343; MATERIAL (none) -> CT; PRICE 1.3 -> 7.60; URL http://www.tme.eu/cz/details/uvz1c101mdd/elektrolyticke-kon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 -> http://www.tme.eu/cz/details/293d226x9025d2te3/tantalove-ko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; VOLTAGE 16V -> 25V
- C4: value 22p -> 1000M; device !discrete:C0805 -> !discrete:CE_D10L13_L; MATERIAL (none) -> CE; PRICE 0.16 -> 1.80; URL http://www.tme.eu/cz/details/cc0805krx7r9104/kondenzatory-m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 -> http://www.tme.eu/cz/details/pf1a102mnn1016/elektrolyticke-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; VOLTAGE 16V -> 6V3
- C6: value 22p -> 1000M; device !discrete:C0805 -> !discrete:CE_D10L13_R; MATERIAL (none) -> CE; PRICE 0.16 -> 1.80; URL http://www.tme.eu/cz/details/cc0805krx7r9104/kondenzatory-m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 -> http://www.tme.eu/cz/details/pf1a102mnn1016/elektrolyticke-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; VOLTAGE 16V -> 6V3
- D2, D4, D5: value G -> KP-2012SGC; PRICE 1 -> (none); URL http://www.tme.eu/cz/details/kp-2012sgc/diody-led-smd-barev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 -> (none)
- D3: value O -> KP-2012SGC; PRICE 1 -> (none); URL http://www.tme.eu/cz/details/kp-2012sgc/diody-led-smd-barev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 -> (none)
- D6: value R -> KP-2012SGC; PRICE 1 -> (none); URL http://www.tme.eu/cz/details/kp-2012sgc/diody-led-smd-barev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 -> (none)
- D7: PRICE (none) -> 0.50; URL (none) -> http://www.tme.eu/cz/details/ll4148-dio/univerzalni-diody-s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
- D8: value BZV55C3.3 -> BZV55C3V3; PRICE (none) -> 0.70; URL (none) -> http://www.tme.eu/cz/details/bzv55c3v3/zenerovy-diody-smd/d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
- D9: value BZV55V3.3 -> BZV55C3V3; PRICE (none) -> 0.70; URL (none) -> http://www.tme.eu/cz/details/bzv55c3v3/zenerovy-diody-smd/d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
- IO2: PRICE 228.35 -> 63.50; URL http://www.tme.eu/cz/details/ds3234sn/pameti-sram-paralelni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 -> https://www.aliexpress.com/item/100-new-original-DS3234SN-T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
- JP1: value S2G3_JUM -> DS1021-1*8SF1-1; device #Lamacie lišty by TD:S2G3_JUM -> !pinhead:PINHD-1X7; PRICE (none) -> 1.60; URL (none) -> http://www.tme.eu/cz/details/zl201-08g/konektory-hrebinky/c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
- JP10, JP4, JP7, JP8, JP9: value S1G3_JUM -> DS1021-1*8SF1-1; device #Lamacie lišty by TD:S1G3_JUM -> !pinhead:PINHD-1X8; PRICE (none) -> 1.60; URL (none) -> http://www.tme.eu/cz/details/zl201-08g/konektory-hrebinky/c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
- JP11, JP2, JP3: value S1G3_JUM -> DS1021-1*8SF1-1; device #Lamacie lišty by TD:S1G3_JUM -> !pinhead:PINHD-1X7; PRICE (none) -> 1.60; URL (none) -> http://www.tme.eu/cz/details/zl201-08g/konektory-hrebinky/c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
- JP5: value S1G8_JUM -> DS1021-1*8SF1-1; device #Lamacie lišty by TD:S1G8_JUM -> !pinhead:PINHD-1X8; PRICE (none) -> 1.60; URL (none) -> http://www.tme.eu/cz/details/zl201-08g/konektory-hrebinky/c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
- JP6: value S1G2_JUM -> DS1021-1*8SF1-1; device #Lamacie lišty by TD:S1G2_JUM -> !pinhead:PINHD-1X7; PRICE (none) -> 1.60; URL (none) -> http://www.tme.eu/cz/details/zl201-08g/konektory-hrebinky/c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
- R1, R11, R3, R7: value 470R -> 330; PRICE 0.5 -> 0.15; TOLERANCE 1% -> (none); URL http://www.tme.eu/cz/details/hp05-470r1%25/rezistory-smd-08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 -> http://www.tme.eu/cz/details/smd0805-330r/rezistory-smd-080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
- R10: value 330R -> 330
- R12, R14, R16, R17, R18, R19, R2, R4, R8: value 330R -> 330; PRICE 0.22 -> 0.15; TOLERANCE 1% -> (none); URL http://www.tme.eu/cz/details/smd0805-330r-1%25/rezistory-sm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 -> http://www.tme.eu/cz/details/smd0805-330r/rezistory-smd-080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
- R13: value 10k -> *; PRICE 0.15 -> (none); TOLERANCE 5% -> (none); URL http://www.tme.eu/cz/details/rc0805jr-07510k/rezistory-smd-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 -> (none)
- R6: value 10k -> 330; PRICE 0.15 -> 0.22; TOLERANCE 5% -> 1%; URL http://www.tme.eu/cz/details/rc0805jr-07510k/rezistory-smd-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 -> http://www.tme.eu/cz/details/smd0805-330r-1%25/rezistory-sm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
- R9: value 10k -> 100k; PRICE 0.15 -> 0.22; TOLERANCE 5% -> 1%; URL http://www.tme.eu/cz/details/rc0805jr-07510k/rezistory-smd-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 -> http://www.tme.eu/cz/details/smd0805-100k-1%25/rezistory-sm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
- SW1, SW2: PRICE 18 -> 17.00; URL https://www.gme.cz/tlacitkovy-spinac-p-dt6rt -> http://www.tme.eu/cz/details/d6r-b/mikrospinace-tact-pcb/ck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
- T2: value (none) -> IRLML0060; PRICE (none) -> 3.00; URL (none) -> http://www.tme.eu/cz/details/irlml0060trpbf/tranzistory-s-k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
Connections:
- removed net ECHO1-PD7: IO1A.PD7(AIN1), R11.2, R12.2
- removed net ECHO2-PB0: IO1A.PB0(ICP), R3.2, R4.2
- removed net ECHO3-PB3: IO1A.PB3(MOSI/OC2), JP1G$1.2, R1.2, R2.2
- removed net ECHO4-PB4: IO1A.PB4(MISO), JP1G$2.3, R7.2, R8.2
- removed net GPA0-2: IO4.GPA0, JP14.1
- removed net GPA1-2: IO4.GPA1, JP14.2
- removed net GPA2-2: IO4.GPA2, JP14.3
- removed net GPA3-2: IO4.GPA3, JP14.4
- removed net GPA4-2: IO4.GPA4, JP14.5
- removed net GPA5-2: IO4.GPA5, JP14.6
- removed net GPA6-2: IO4.GPA6, JP14.7
- removed net GPA7-2: IO4.GPA7, JP14.8
- removed net GPB0-2: IO4.GPB0, R16.1
- removed net GPB1-2: IO4.GPB1, R18.1
- removed net GPB2-2: IO4.GPB2, R14.1
- removed net GPB3-2: IO4.GPB3, R17.1
- removed net GPB4-2: IO4.GPB4, R19.1
- removed net GPB5-2: IO4.GPB5, R20.1, SW1.2, SW1.4
- removed net GPB6-2: IO4.GPB6, R21.1, SW2.2, SW2.4
- removed net GPB7-2: IO4.GPB7, R15.1
- removed net INT/SQW: IO2.INT/SQW
- removed net INTA1: IO4.INTA, JP6.2
- removed net INTB1: IO4.INTB, JP6.1
- removed net N$1: JP11.3, R8.1
- removed net N$11: JP3.3, R12.1
- removed net N$23: D1.A, R10.1
- removed net N$5: JP10.3, R2.1
- removed net N$8: JP7.3, R4.1
- removed net RESET: IO1A.PC6/#RESET, JP1G$2.1, R13.2
- removed net SCK: IO1A.PB5(SCK), JP1G$2.2
- removed net TRIG1-PD5-OC0B: IO1A.PD5(T1), JP2.1
- removed net TRIG2-PD6-OC0A: IO1A.PD6(AIN0), JP4.1
- removed net TRIG3-PB1-OC1A: IO1A.PB1(OC1A), JP8.1
- removed net TRIG4-PB2-OC1B: IO1A.PB2(SS/OC1B), JP9.1
- removed net XTAL1: C4.2, IO1A.PB6/XTAL1, Q1.2
- removed net XTAL2: C6.2, IO1A.PB7/XTAL2, Q1.1
- new net INT: IC2.INTA, IC2.INTB, R9.2, RPI.GPIO4/GCKL
- new net LED0: IC1.LED0, IC3.I7
- new net N$17: IC1.LED1, IC3.I6
- new net N$18: D10.A, D11.A, D12.A, D13.A, D14.A, D15.A, D16.A, IC3.CD+, JP1.1, JP1.2, JP1.3, JP1.4, JP1.5, JP1.6, JP1.7, R13.2
- new net N$19: IC1.LED2, IC3.I5
- new net N$20: D10.C, R1.2
- new net N$21: D16.C, R11.2
- new net N$24: IC1.LED4, IC3.I4
- new net N$25: IC1.LED5, IC3.I3
- new net N$26: IC1.LED6, IC3.I2
- new net N$27: IC1.LED7, IC3.I1
- new net N$28: D15.C, R8.2
- new net N$29: D14.C, R7.2
- new net N$30: D13.C, R4.2
- new net N$31: D12.C, R3.2
- new net N$32: D11.C, R2.2
- new net N$33: D5.C, R17.2
- new net N$34: D4.C, R16.2
- new net N$35: D3.C, R14.2
- new net N$37: D19.C, R23.2
- new net N$38: D25.C, R29.2
- new net N$39: D24.C, R28.2
- new net N$40: D23.C, R27.2
- new net N$41: D22.C, R26.2
- new net N$42: D21.C, R25.2
- new net N$43: D20.C, R24.2
- new net N$9: D27.A, R6.1
- new net PA0: IC2.GPA0, JP10.8, R12.1
- new net PA1: IC2.GPA1, JP10.7, R14.1
- new net PA2: IC2.GPA2, JP10.6, R16.1
- new net PA3: IC2.GPA3, JP10.5, R17.1
- new net PA4: IC2.GPA4, JP10.4, R18.1
- new net PA5: IC2.GPA5, JP10.3, R19.1
- new net PA6: IC2.GPA6, JP10.2, R20.1, R22.1, SW1.2, SW1.4
- new net PA7: IC2.GPA7, JP10.1, R21.1, R30.1, SW2.2, SW2.4
- new net PB0: IC2.GPB0, JP6.7, R23.1
- new net PB1: IC2.GPB1, JP6.6, R24.1
- new net PB2: IC2.GPB2, JP6.5, R25.1
- new net PB3: IC2.GPB3, JP6.4, R26.1
- new net PB4: IC2.GPB4, JP6.3, R27.1
- new net PB5: IC2.GPB5, JP6.2, R28.1
- new net PB6: IC2.GPB6, JP6.1, R29.1
- new net PB7: IC2.GPB7, R15.1
- new net PWM0: IC3.O7, JP2.1, R1.1
- new net PWM1: IC3.O6, JP2.2, R2.1
- new net PWM2: IC3.O5, JP2.3, R3.1
- new net PWM4: IC3.O4, JP2.4, R4.1
- new net PWM5: IC3.O3, JP2.7, R11.1
- new net PWM6: IC3.O2, JP2.5, R7.1
- new net PWM7: IC3.O1, JP2.6, R8.1
- net +3V3: now also C12.1, C4.+, D1.A, D17.A, D18.A, D19.A, D2.A, D20.A, D21.A, D22.A, D23.A, D24.A, D25.A, D26.A, D3.A, D4.A, D5.A, D6.A, IC1.VDD, IC2.!RESET, IC2.VDD, IC4.OUT, JP11.1, JP11.2, JP11.3, JP11.4, JP11.5, JP11.6, JP11.7, JP7.1, JP7.2, JP7.3, JP7.4, JP7.5, JP7.6, JP7.7, JP7.8, JP8.1, JP8.2, JP8.3, JP8.4, JP8.5, JP8.6, JP8.7, JP8.8, R9.1; no longer C3.+, IO1A.ADC6, IO1A.ADC7, IO1A.AREF, IO1A.PC0(ADC0), IO1A.PC1(ADC1), IO1A.PC2(ADC2), IO1A.PC3(ADC3), IO1A.PD0(RXD), IO1A.PD1(TXD), IO1A.PD2(INT0), IO1A.PD3(INT1), IO1A.PD4(XCK/T0), IO1AP.VCC, IO1P1.VCC, IO1P2.VCC, IO4.!RESET, IO4.VDD, IO5.OUT, JP1G$1.3, JP24.1, JP24.2, JP24.3, JP24.4, JP24.5, JP24.6, JP24.7, JP24.8, JP29.1, JP29.2, JP29.3, JP29.4, JP29.5, JP29.6, JP29.7, JP29.8, R10.2, R13.1, R9.2
- net +5V: now also C6.+, IC4.IN, R13.1, R6.2; no longer C1.+, IO5.IN, JP10.2, JP11.2, JP2.2, JP3.2, JP4.2, JP7.2, JP8.2, JP9.2
- net AD0: now also JP4.8; no longer JP5.1
- net AD1: now also JP4.1; no longer JP5.8
- net AD2: now also JP4.7; no longer JP5.2
- net AD3: now also JP4.2; no longer JP5.7
- net AD4: now also JP4.6; no longer JP5.3
- net AD5: now also JP4.3; no longer JP5.6
- net AD6: now also JP4.5; no longer JP5.4
- net AD7: now also JP4.4; no longer JP5.5
- net AGND: now also IO3.AS, JP5.1, JP5.2, JP5.3, JP5.4, JP5.5, JP5.6, JP5.7, JP5.8; no longer JP28.1, JP28.2, JP28.3, JP28.4, JP28.5, JP28.6, JP28.7, JP28.8, R6.2
- net GND: now also C1.2, C11.-, C12.2, C4.-, C6.-, D27.C, D28.A, IC1.A0, IC1.A1, IC1.A2, IC1.A3, IC1.A4, IC1.A5, IC1.CLK, IC1.OE, IC1.VSS, IC2.A0, IC2.A1, IC2.A2, IC2.VSS, IC3.GND, IC4.GND, JP12.1, JP12.2, JP12.3, JP12.4, JP12.5, JP12.6, JP12.7, JP13.1, JP3.2, JP3.3, JP3.4, JP3.5, JP3.6, JP3.7, JP9.1, JP9.2, JP9.4, JP9.5, JP9.6, JP9.7, JP9.8, R10.1; no longer ARK1.K1, C1.-, C4.1, C6.1, D1.C, D2.C, D3.C, D4.C, D5.C, D6.C, IO1AP.GND, IO1P1.GND, IO1P2.GND, IO4.A0, IO4.A1, IO4.A2, IO4.VSS, IO5.GND, JP10.1, JP11.1, JP1G$1.1, JP2.3, JP23.1, JP23.2, JP23.3, JP23.4, JP23.5, JP23.6, JP23.7, JP23.8, JP4.3, JP7.1, JP8.3, R1.1, R11.1, R3.1, R7.1
- net N$12: now also C1.1, C11.+, C3.+, D28.K
- net N$16: now also JP13.2; no longer ARK1.K2
- net N$2: now also D26.C, R30.2; no longer D6.A, R19.2
- net N$22: now also D1.C, R10.2; no longer IO3.AS, R6.1, R9.1
- net N$3: now also D2.C, R12.2; no longer D3.A, R17.2
- net N$4: now also D18.C, R22.2; no longer D4.A, R14.2
- net N$6: now also D17.C, R19.2; no longer D5.A, R18.2
- net N$7: now also D6.C, R18.2; no longer D2.A, R16.2
- net SCL: now also IC1.SCL, IC2.SCL; no longer IO1A.PC5(SCL/ADC5), IO4.SCL
- net SDA: now also IC1.SDA, IC2.SDA; no longer IO1A.PC4(SDA/ADC4), IO4.SDA
Other:
- note added: "ADC adresa na I2C 0x21"
- note added: "PWM adresa na I2C 0x40"
- note removed: "Urcuje Adresu I2C"
- note removed: "adresa 0x21 musi byt odpor"
- note removed: "adresa 0x22 musi byt odpor"

Commit message: KM2 a MAINBOARD - posledni upravy pred Release
Parts:
- removed IO2: DS3234, SparkFun:DS3234
- added IC5: DS3234, !ic_maxim:DS3234
Connections:
- net +3V3: now also IC5.VCC; no longer IO2.VCC
- net CE0: now also IC5.CS; no longer IO2.CS
- net GND: now also IC5.GND, IC5.GND@10, IC5.GND@11, IC5.GND@12, IC5.GND@13, IC5.GND@14, IC5.GND@2, IC5.GND@7, IC5.GND@8, IC5.GND@9; no longer IO2.GND, IO2.GND@10, IO2.GND@11, IO2.GND@12, IO2.GND@13, IO2.GND@14, IO2.GND@2, IO2.GND@7, IO2.GND@8, IO2.GND@9
- net MISO: now also IC5.DOUT; no longer IO2.DOUT
- net MOSI: now also IC5.DIN; no longer IO2.DIN
- net SCLK: now also IC5.SCLK@18, IC5.SCLK@20; no longer IO2.SCLK@18, IO2.SCLK@20
- net VBATT: now also IC5.VBAT; no longer IO2.VBAT
